File: system-board/button-ports.kicad_sch (KiCad schematic)
At the start: 3 parts, among them J9 BTNS

Commit message: First attempt
Parts:
- J9: value BTNS -> BTNs; footprint Connector_JST:JST_SH_SM05B-SRSS-TB_1x05-1MP_P1.00mm_Horizontal -> Connector_PinSocket_2.00mm:PinSocket_2x03_P2.00mm_Vertical; symbol Connector:Conn_01x05_Socket -> Connector_Generic:Conn_02x03_Odd_Even
Connections:
- net BTN1: now also J9.3 (Pin_3); no longer J9.2 (Pin_2)
- net BTN2: now also J9.4 (Pin_4); no longer J9.5 (Pin_5)
- net GND: now also J9.2 (Pin_2)
- net at R21.1: now also J9.5 (Pin_5); no longer J9.3 (Pin_3)
- net at R22.1: now also J9.6 (Pin_6); no longer J9.4 (Pin_4)
Other:
- moved on the sheet: J9, R22
Changed lines of the file:
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@@
 (kicad_sch (version 20230121) (generator eeschema)
   (paper "A4")
-  (wire (pts (xy 140.97 78.74) (xy 156.21 78.74))
-    (stroke (width 0) (type default))
-  )
-  (wire (pts (xy 138.43 71.12) (xy 138.43 81.28))
+  (wire (pts (xy 133.35 50.8) (xy 118.11 50.8))
     (stroke (width 0) (type default))
   )
@@
     (stroke (width 0) (type default))
   )
+  (wire (pts (xy 125.73 53.34) (xy 130.81 53.34))
+    (stroke (width 0) (type default))
+  )
   (wire (pts (xy 114.3 78.74) (xy 133.35 78.74))
     (stroke (width 0) (type default))
   )
-  (wire (pts (xy 133.35 78.74) (xy 133.35 71.12))
+  (wire (pts (xy 135.89 71.12) (xy 135.89 81.28))
     (stroke (width 0) (type default))
   )
@@
     (stroke (width 0) (type default))
   )
-  (wire (pts (xy 135.89 71.12) (xy 135.89 81.28))
-    (stroke (width 0) (type default))
-  )
-  (wire (pts (xy 140.97 78.74) (xy 140.97 71.12))
+  (wire (pts (xy 133.35 50.8) (xy 133.35 58.42))
     (stroke (width 0) (type default))
   )
@@
     (stroke (width 0) (type default))
   )
-  (wire (pts (xy 138.43 81.28) (xy 143.51 81.28))
+  (wire (pts (xy 135.89 48.26) (xy 130.81 48.26))
+    (stroke (width 0) (type default))
+  )
+  (wire (pts (xy 135.89 48.26) (xy 135.89 58.42))
     (stroke (width 0) (type default))
   )
@@
     (stroke (width 0) (type default))
   )
-  (wire (pts (xy 151.13 81.28) (xy 156.21 81.28))
+  (wire (pts (xy 133.35 71.12) (xy 133.35 78.74))
+    (stroke (width 0) (type default))
+  )
+  (wire (pts (xy 130.81 53.34) (xy 130.81 58.42))
+    (stroke (width 0) (type default))
+  )
+  (wire (pts (xy 123.19 48.26) (xy 118.11 48.26))
     (stroke (width 0) (type default))
   )
@@
     (effects (font (size 1.27 1.27)) (justify right))
   )
-  (hierarchical_label "BTN2" (shape passive) (at 156.21 78.74 0) (fields_autoplaced)
-    (effects (font (size 1.27 1.27)) (justify left))
+  (hierarchical_label "BTN2" (shape passive) (at 118.11 50.8 180) (fields_autoplaced)
+    (effects (font (size 1.27 1.27)) (justify right))
   )
   (hierarchical_label "BTN1" (shape passive) (at 114.3 78.74 180) (fields_autoplaced)
     (effects (font (size 1.27 1.27)) (justify right))
   )
-  (hierarchical_label "LED2" (shape passive) (at 156.21 81.28 0) (fields_autoplaced)
-    (effects (font (size 1.27 1.27)) (justify left))
-  )
-  (symbol (lib_id "Connector:Conn_01x05_Socket") (at 135.89 66.04 90) (unit 1)
-    (in_bom yes) (on_board yes) (dnp no) (fields_autoplaced)
-    (property "Reference" "J9" (at 135.89 60.96 90)
+  (hierarchical_label "LED2" (shape passive) (at 118.11 48.26 180) (fields_autoplaced)
+    (effects (font (size 1.27 1.27)) (justify right))
+  )
+  (symbol (lib_id "Connector_Generic:Conn_02x03_Odd_Even") (at 133.35 66.04 90) (unit 1)
+    (in_bom yes) (on_board yes) (dnp no) (fields_autoplaced)
+    (property "Reference" "J9" (at 133.35 60.96 90)
       (effects (font (size 1.27 1.27)))
     )
-    (property "Value" "BTNS" (at 135.89 63.5 90)
+    (property "Value" "BTNs" (at 133.35 63.5 90)
       (effects (font (size 1.27 1.27)))
     )
-    (property "Footprint" "Connector_JST:JST_SH_SM05B-SRSS-TB_1x05-1MP_P1.00mm_Horizontal" (at 135.89 66.04 0)
-      (effects (font (size 1.27 1.27)) hide)
-    )
-    (property "Datasheet" "~" (at 135.89 66.04 0)
+    (property "Footprint" "Connector_PinSocket_2.00mm:PinSocket_2x03_P2.00mm_Vertical" (at 133.35 66.04 0)
+      (effects (font (size 1.27 1.27)) hide)
+    )
+    (property "Datasheet" "~" (at 133.35 66.04 0)
       (effects (font (size 1.27 1.27)) hide)
     )
@@
     (pin "4")
     (pin "5")
+    (pin "6")
     (instances
       (project "system-board"
@@
     )
   )
-  (symbol (lib_id "Device:R_US") (at 147.32 81.28 90) (unit 1)
-    (in_bom yes) (on_board yes) (dnp no) (fields_autoplaced)
-    (property "Reference" "R22" (at 146.05 83.82 0)
-      (effects (font (size 1.27 1.27)) (justify right))
-    )
-    (property "Value" "1k" (at 148.59 83.82 0)
-      (effects (font (size 1.27 1.27)) (justify right))
-    )
-    (property "Footprint" "Resistor_SMD:R_0402_1005Metric" (at 147.574 80.264 90)
-      (effects (font (size 1.27 1.27)) hide)
-    )
-    (property "Datasheet" "https://www.mouser.com/datasheet/2/418/3/NG_CS_1309350_PASSIVE_COMPONENT_0807-1235596.pdf" (at 147.32 81.28 0)
-      (effects (font (size 1.27 1.27)) hide)
-    )
-    (property "JLCPCB Part #" "C2073750" (at 147.32 81.28 0)
-      (effects (font (size 1.27 1.27)) hide)
-    )
-    (property "Manufacturer" "TE Connectivity" (at 147.32 81.28 0)
-      (effects (font (size 1.27 1.27)) hide)
-    )
-    (property "Manufacturer_Part_Number" "CRG0402F1K0" (at 147.32 81.28 0)
-      (effects (font (size 1.27 1.27)) hide)
-    )
-    (property "Mouser Part Number" "279-CRG0402F1K0 " (at 147.32 81.28 0)
+  (symbol (lib_id "Device:R_US") (at 127 48.26 270) (unit 1)
+    (in_bom yes) (on_board yes) (dnp no) (fields_autoplaced)
+    (property "Reference" "R22" (at 128.27 45.72 0)
+      (effects (font (size 1.27 1.27)) (justify right))
+    )
+    (property "Value" "1k" (at 125.73 45.72 0)
+      (effects (font (size 1.27 1.27)) (justify right))
+    )
+    (property "Footprint" "Resistor_SMD:R_0402_1005Metric" (at 126.746 49.276 90)
+      (effects (font (size 1.27 1.27)) hide)
+    )
+    (property "Datasheet" "https://www.mouser.com/datasheet/2/418/3/NG_CS_1309350_PASSIVE_COMPONENT_0807-1235596.pdf" (at 127 48.26 0)
+      (effects (font (size 1.27 1.27)) hide)
+    )
+    (property "JLCPCB Part #" "C2073750" (at 127 48.26 0)
+      (effects (font (size 1.27 1.27)) hide)
+    )
+    (property "Manufacturer" "TE Connectivity" (at 127 48.26 0)
+      (effects (font (size 1.27 1.27)) hide)
+    )
+    (property "Manufacturer_Part_Number" "CRG0402F1K0" (at 127 48.26 0)
+      (effects (font (size 1.27 1.27)) hide)
+    )
+    (property "Mouser Part Number" "279-CRG0402F1K0 " (at 127 48.26 0)
       (effects (font (size 1.27 1.27)) hide)
     )
@@
         )
       )
+    )
+  )
+  (symbol (lib_id "power:GND") (at 125.73 53.34 270) (unit 1)
+    (in_bom yes) (on_board yes) (dnp no) (fields_autoplaced)
+    (property "Reference" "#PWR043" (at 119.38 53.34 0)
+      (effects (font (size 1.27 1.27)) hide)
+    )
+    (property "Value" "GND" (at 121.92 53.34 90)
+      (effects (font (size 1.27 1.27)) (justify right))
+    )
+    (property "Footprint" "" (at 125.73 53.34 0)
+      (effects (font (size 1.27 1.27)) hide)
+    )
+    (property "Datasheet" "" (at 125.73 53.34 0)
+      (effects (font (size 1.27 1.27)) hide)
+    )
+    (pin "1")
+    (instances
+      (project "system-board"
+        (path "/54f22c46-3801-43f0-a916-fc0a05246fe7/3781b295-d7aa-4373-9a43-be57335904e5"
+          (reference "#PWR043") (unit 1)
+        )
+      )

Commit message: Redo system-board PCB to use fewer connectors
Parts:
- J9: now left out of the parts list
- R21, R22: digikey part number (none) -> A121534TR-ND
Changed lines of the file:
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@@
   )
   (symbol (lib_id "Connector_Generic:Conn_02x03_Odd_Even") (at 133.35 66.04 90) (unit 1)
-    (in_bom yes) (on_board yes) (dnp no) (fields_autoplaced)
+    (in_bom no) (on_board yes) (dnp no) (fields_autoplaced)
     (property "Reference" "J9" (at 133.35 60.96 90)
       (effects (font (size 1.27 1.27)))
@@
     )
     (property "Mouser Part Number" "279-CRG0402F1K0 " (at 127 48.26 0)
+      (effects (font (size 1.27 1.27)) hide)
+    )
+    (property "digikey part number" "A121534TR-ND" (at 127 48.26 0)
       (effects (font (size 1.27 1.27)) hide)
     )
@@
       (effects (font (size 1.27 1.27)) hide)
     )
+    (property "digikey part number" "A121534TR-ND" (at 124.46 81.28 0)
+      (effects (font (size 1.27 1.27)) hide)
+    )

Commit message: Yet another PCB Revision
Parts:
- J9: now not fitted
- R21, R22: MPN (none) -> CRG0402F1K0; package (none) -> 0402
Changed lines of the file:
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@@
   )
   (symbol (lib_id "Connector_Generic:Conn_02x03_Odd_Even") (at 133.35 66.04 90) (unit 1)
-    (in_bom no) (on_board yes) (dnp no) (fields_autoplaced)
+    (in_bom no) (on_board yes) (dnp yes) (fields_autoplaced)
     (property "Reference" "J9" (at 133.35 60.96 90)
       (effects (font (size 1.27 1.27)))
@@
     )
     (property "Datasheet" "~" (at 133.35 66.04 0)
+      (effects (font (size 1.27 1.27)) hide)
+    )
+    (property "MPN" "" (at 133.35 66.04 0)
       (effects (font (size 1.27 1.27)) hide)
     )
@@
     )
     (property "digikey part number" "A121534TR-ND" (at 127 48.26 0)
+      (effects (font (size 1.27 1.27)) hide)
+    )
+    (property "package" "0402" (at 127 48.26 0)
+      (effects (font (size 1.27 1.27)) hide)
+    )
+    (property "MPN" "CRG0402F1K0" (at 127 48.26 0)
       (effects (font (size 1.27 1.27)) hide)
     )
@@
       (effects (font (size 1.27 1.27)) hide)
     )
+    (property "package" "0402" (at 124.46 81.28 0)
+      (effects (font (size 1.27 1.27)) hide)
+    )
+    (property "MPN" "CRG0402F1K0" (at 124.46 81.28 0)
+      (effects (font (size 1.27 1.27)) hide)
+    )

Commit message: Redo design again
Parts:
- renumbered J9 to J6, R22 to R16, R21 to R17
Changed lines of the file:
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@@
   (symbol (lib_id "Connector_Generic:Conn_02x03_Odd_Even") (at 133.35 66.04 90) (unit 1)
     (in_bom no) (on_board yes) (dnp yes) (fields_autoplaced)
-    (property "Reference" "J9" (at 133.35 60.96 90)
+    (property "Reference" "J6" (at 133.35 60.96 90)
       (effects (font (size 1.27 1.27)))
     )
@@
       (project "system-board"
         (path "/54f22c46-3801-43f0-a916-fc0a05246fe7/3781b295-d7aa-4373-9a43-be57335904e5"
-          (reference "J9") (unit 1)
+          (reference "J6") (unit 1)
         )
       )
@@
   (symbol (lib_id "Device:R_US") (at 127 48.26 270) (unit 1)
     (in_bom yes) (on_board yes) (dnp no) (fields_autoplaced)
-    (property "Reference" "R22" (at 128.27 45.72 0)
+    (property "Reference" "R16" (at 128.27 45.72 0)
       (effects (font (size 1.27 1.27)) (justify right))
     )
@@
       (project "system-board"
         (path "/54f22c46-3801-43f0-a916-fc0a05246fe7/3781b295-d7aa-4373-9a43-be57335904e5"
-          (reference "R22") (unit 1)
+          (reference "R16") (unit 1)
         )
       )
@@
   (symbol (lib_id "power:GND") (at 125.73 76.2 270) (unit 1)
     (in_bom yes) (on_board yes) (dnp no) (fields_autoplaced)
-    (property "Reference" "#PWR058" (at 119.38 76.2 0)
+    (property "Reference" "#PWR049" (at 119.38 76.2 0)
       (effects (font (size 1.27 1.27)) hide)
     )
@@
       (project "system-board"
         (path "/54f22c46-3801-43f0-a916-fc0a05246fe7/3781b295-d7aa-4373-9a43-be57335904e5"
-          (reference "#PWR058") (unit 1)
+          (reference "#PWR049") (unit 1)
         )
       )
@@
   (symbol (lib_id "Device:R_US") (at 124.46 81.28 270) (mirror x) (unit 1)
     (in_bom yes) (on_board yes) (dnp no) (fields_autoplaced)
-    (property "Reference" "R21" (at 125.73 83.82 0)
+    (property "Reference" "R17" (at 125.73 83.82 0)
       (effects (font (size 1.27 1.27)) (justify right))
     )
@@
       (project "system-board"
         (path "/54f22c46-3801-43f0-a916-fc0a05246fe7/3781b295-d7aa-4373-9a43-be57335904e5"
-          (reference "R21") (unit 1)
+          (reference "R17") (unit 1)
         )
       )
@@
   (symbol (lib_id "power:GND") (at 125.73 53.34 270) (unit 1)
     (in_bom yes) (on_board yes) (dnp no) (fields_autoplaced)
-    (property "Reference" "#PWR043" (at 119.38 53.34 0)
+    (property "Reference" "#PWR048" (at 119.38 53.34 0)
       (effects (font (size 1.27 1.27)) hide)
     )
@@
       (project "system-board"
         (path "/54f22c46-3801-43f0-a916-fc0a05246fe7/3781b295-d7aa-4373-9a43-be57335904e5"
-          (reference "#PWR043") (unit 1)
+          (reference "#PWR048") (unit 1)
         )
       )
