File: system-board/i2s_amp.kicad_sch (KiCad schematic)
At the start: 9 parts, among them J2 SPKR, U1 MAX98357AETE+T

Commit message: First attempt
Parts:
- J2: footprint Connector_JST:JST_SH_SM02B-SRSS-TB_1x02-1MP_P1.00mm_Horizontal -> Connector_PinSocket_2.00mm:PinSocket_1x02_P2.00mm_Vertical
- U1: footprint MaximCustom:Maxim_Integrated-T1633-4-0-V-IPC_C -> Imports:Maxim_Integrated-T1633-4-0-V-IPC_C
Changed lines of the file:
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@@
       (effects (font (size 1.27 1.27)))
     )
-    (property "Footprint" "MaximCustom:Maxim_Integrated-T1633-4-0-V-IPC_C" (at 168.91 107.95 0)
+    (property "Footprint" "Imports:Maxim_Integrated-T1633-4-0-V-IPC_C" (at 168.91 107.95 0)
       (effects (font (size 1.27 1.27)) (justify left) hide)
     )
@@
       (effects (font (size 1.27 1.27)))
     )
-    (property "Footprint" "Connector_JST:JST_SH_SM02B-SRSS-TB_1x02-1MP_P1.00mm_Horizontal" (at 87.63 99.06 0)
+    (property "Footprint" "Connector_PinSocket_2.00mm:PinSocket_1x02_P2.00mm_Vertical" (at 87.63 99.06 0)
       (effects (font (size 1.27 1.27)) hide)
     )

Commit message: Redo system-board PCB to use fewer connectors
Parts:
- C1: digikey part number (none) -> 490-GRM155R60J106ME05DTR-ND
- C2: digikey part number (none) -> 399-C0402C104K9RAC7867TR-ND
- C3, C4: digikey part number (none) -> 732-8048-2-ND
- FB1, FB2: digikey part number (none) -> MH1608-471YTR-ND
- R1: digikey part number (none) -> A130391TR-ND
- U1: Manufacturer_Part_Number (none) -> MAX98357AETE+T; Mouser Part Number (none) -> 700-MAX98357AETE+T; automotive No -> (none); manufacturer Maxim Integrated -> (none); power at speaker r 3.2W @ 4Ω -> (none); voltage gain 15dB -> (none)
Changed lines of the file:
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@@
+      (effects (font (size 1.27 1.27)) hide)
+    )
+    (property "digikey part number" "399-C0402C104K9RAC7867TR-ND" (at 161.29 113.03 0)
       (effects (font (size 1.27 1.27)) hide)
     )
@@
       (effects (font (size 1.27 1.27)) hide)
     )
+    (property "digikey part number" "732-8048-2-ND" (at 105.41 83.82 0)
+      (effects (font (size 1.27 1.27)) hide)
+    )
     (pin "1")
     (pin "2")
@@
       (effects (font (size 1.27 1.27)) hide)
     )
+    (property "digikey part number" "MH1608-471YTR-ND" (at 116.84 95.25 0)
+      (effects (font (size 1.27 1.27)) hide)
+    )
     (pin "1")
     (pin "2")
@@
       (effects (font (size 1.27 1.27)) (justify left) hide)
     )
-    (property "automotive" "No" (at 168.91 113.03 0)
-      (effects (font (size 1.27 1.27)) (justify left) hide)
-    )
     (property "category" "IC" (at 168.91 115.57 0)
       (effects (font (size 1.27 1.27)) (justify left) hide)
@@
       (effects (font (size 1.27 1.27)) (justify left) hide)
     )
-    (property "manufacturer" "Maxim Integrated" (at 168.91 143.51 0)
-      (effects (font (size 1.27 1.27)) (justify left) hide)
-    )
     (property "max junction temp" "+150°C" (at 168.91 146.05 0)
       (effects (font (size 1.27 1.27)) (justify left) hide)
@@
       (effects (font (size 1.27 1.27)) (justify left) hide)
     )
-    (property "power at speaker r" "3.2W @ 4Ω" (at 168.91 163.83 0)
-      (effects (font (size 1.27 1.27)) (justify left) hide)
-    )
     (property "rohs" "Yes" (at 168.91 166.37 0)
       (effects (font (size 1.27 1.27)) (justify left) hide)
@@
       (effects (font (size 1.27 1.27)) (justify left) hide)
     )
-    (property "voltage gain" "15dB" (at 168.91 176.53 0)
-      (effects (font (size 1.27 1.27)) (justify left) hide)
-    )
     (property "JLCPCB Part #" "C910544" (at 168.91 97.79 0)
       (effects (font (size 1.27 1.27)) hide)
@@
     )
     (property "Substitution Comments" "Need to keep this compatible." (at 168.91 97.79 0)
+      (effects (font (size 1.27 1.27)) hide)
+    )
+    (property "Manufacturer_Part_Number" "MAX98357AETE+T " (at 168.91 97.79 0)
+      (effects (font (size 1.27 1.27)) hide)
+    )
+    (property "Mouser Part Number" "700-MAX98357AETE+T" (at 168.91 97.79 0)
       (effects (font (size 1.27 1.27)) hide)
     )
@@
       (effects (font (size 1.27 1.27)) hide)
     )
+    (property "digikey part number" "490-GRM155R60J106ME05DTR-ND" (at 161.29 107.95 0)
+      (effects (font (size 1.27 1.27)) hide)
+    )
     (pin "1")
     (pin "2")
@@
     )
     (property "Mouser Part Number" "279-CRGP0402F1M0" (at 171.45 93.98 0)
+      (effects (font (size 1.27 1.27)) hide)
+    )
+    (property "digikey part number" "A130391TR-ND" (at 171.45 93.98 0)
       (effects (font (size 1.27 1.27)) hide)
     )
@@
       (effects (font (size 1.27 1.27)) hide)
     )
+    (property "digikey part number" "732-8048-2-ND" (at 100.33 83.82 0)
+      (effects (font (size 1.27 1.27)) hide)
+    )
     (pin "1")
     (pin "2")
@@
       (effects (font (size 1.27 1.27)) hide)
     )
+    (property "digikey part number" "MH1608-471YTR-ND" (at 116.84 100.33 0)
+      (effects (font (size 1.27 1.27)) hide)
+    )

Commit message: Yet another PCB Revision
Parts:
- C1: MPN (none) -> GRM155R60J106ME05D; Substitution Comments Keep the value correct. -> (none); package (none) -> 0402
- C2: MPN (none) -> C0402C104K9RACTU; package (none) -> 0402
- C3, C4: MPN (none) -> 885012207056; Substitution Comments Keep the value correct. -> (none); package (none) -> 0805
- FB1: package (none) -> 0603
- FB2: MPN HCB1608KF-102T10 -> MH1608-471Y; Substitution Comments Just make sure it can handle 1A. It's for a low-pass filter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 -> (none); package (none) -> 0603
- J2: now not fitted
- R1: MPN (none) -> CRGP0402F1M0; Substitution Comments Keep the value correct. -> (none); package (none) -> 0402
- U1: MPN (none) -> MAX98357AETE+T; Substitution Comments Need to keep this compatible. -> (none); category IC -> (none); device class L1 Integrated Circuits (ICs) -> (none); device class L2 Linear ICs -> (none); device class L3 Amplifiers - Audio -> (none); digikey description IC AMP CLASS D MONO 3.2W 16TQFN -> (none); height 0.8mm -> (none); ipc land pattern name QFN50P300X300X75-16 -> (none); lead free Yes -> (none); library id f761d93c558e3979 -> (none); max junction temp +150°C -> (none); max supply voltage 5.5V -> (none); min supply voltage 2.5V -> (none); mouser part number 700-MAX98357AETE+T -> (none); nominal supply current 2.4-2.75mA -> (none); number of channels 1 -> (none); rohs Yes -> (none); standoff height 0mm -> (none); temperature range high +85°C -> (none); temperature range low -40°C -> (none)
Changed lines of the file:
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@@
-      (effects (font (size 1.27 1.27)) hide)
-    )
-    (property "Substitution Comments" "" (at 161.29 113.03 0)
       (effects (font (size 1.27 1.27)) hide)
     )
@@
     )
     (property "digikey part number" "399-C0402C104K9RAC7867TR-ND" (at 161.29 113.03 0)
+      (effects (font (size 1.27 1.27)) hide)
+    )
+    (property "package" "0402" (at 161.29 113.03 0)
+      (effects (font (size 1.27 1.27)) hide)
+    )
+    (property "MPN" "C0402C104K9RACTU" (at 161.29 113.03 0)
       (effects (font (size 1.27 1.27)) hide)
     )
@@
       (effects (font (size 1.27 1.27)) hide)
     )
-    (property "Substitution Comments" "Keep the value correct." (at 105.41 83.82 0)
-      (effects (font (size 1.27 1.27)) hide)
-    )
     (property "Manufacturer" "Wurth Elektronik " (at 105.41 83.82 0)
       (effects (font (size 1.27 1.27)) hide)
@@
       (effects (font (size 1.27 1.27)) hide)
     )
+    (property "package" "0805" (at 105.41 83.82 0)
+      (effects (font (size 1.27 1.27)) hide)
+    )
+    (property "MPN" "885012207056 " (at 105.41 83.82 0)
+      (effects (font (size 1.27 1.27)) hide)
+    )
     (pin "1")
     (pin "2")
@@
       (effects (font (size 1.27 1.27)) hide)
     )
+    (property "Manufacturer" "Bourns" (at 116.84 95.25 0)
+      (effects (font (size 1.27 1.27)) hide)
+    )
+    (property "Manufacturer_Part_Number" "MH1608-471Y" (at 116.84 95.25 0)
+      (effects (font (size 1.27 1.27)) hide)
+    )
+    (property "Mouser Part Number" "652-MH1608-471Y" (at 116.84 95.25 0)
+      (effects (font (size 1.27 1.27)) hide)
+    )
+    (property "digikey part number" "MH1608-471YTR-ND" (at 116.84 95.25 0)
+      (effects (font (size 1.27 1.27)) hide)
+    )
+    (property "package" "0603" (at 116.84 95.25 0)
+      (effects (font (size 1.27 1.27)) hide)
+    )
     (property "MPN" "MH1608-471Y" (at 116.84 95.25 0)
-      (effects (font (size 1.27 1.27)) hide)
-    )
-    (property "Manufacturer" "Bourns" (at 116.84 95.25 0)
-      (effects (font (size 1.27 1.27)) hide)
-    )
-    (property "Substitution Comments" "" (at 116.84 95.25 0)
-      (effects (font (size 1.27 1.27)) hide)
-    )
-    (property "Manufacturer_Part_Number" "MH1608-471Y" (at 116.84 95.25 0)
-      (effects (font (size 1.27 1.27)) hide)
-    )
-    (property "Mouser Part Number" "652-MH1608-471Y" (at 116.84 95.25 0)
-      (effects (font (size 1.27 1.27)) hide)
-    )
-    (property "digikey part number" "MH1608-471YTR-ND" (at 116.84 95.25 0)
       (effects (font (size 1.27 1.27)) hide)
     )
@@
       (effects (font (size 1.27 1.27)) (justify left) hide)
     )
-    (property "category" "IC" (at 168.91 115.57 0)
-      (effects (font (size 1.27 1.27)) (justify left) hide)
-    )
-    (property "device class L1" "Integrated Circuits (ICs)" (at 168.91 118.11 0)
-      (effects (font (size 1.27 1.27)) (justify left) hide)
-    )
-    (property "device class L2" "Linear ICs" (at 168.91 120.65 0)
-      (effects (font (size 1.27 1.27)) (justify left) hide)
-    )
-    (property "device class L3" "Amplifiers - Audio" (at 168.91 123.19 0)
-      (effects (font (size 1.27 1.27)) (justify left) hide)
-    )
-    (property "digikey description" "IC AMP CLASS D MONO 3.2W 16TQFN" (at 168.91 125.73 0)
-      (effects (font (size 1.27 1.27)) (justify left) hide)
-    )
     (property "digikey part number" "MAX98357AETE+TCT-ND" (at 168.91 128.27 0)
       (effects (font (size 1.27 1.27)) (justify left) hide)
@@
       (effects (font (size 1.27 1.27)) (justify left) hide)
     )
-    (property "height" "0.8mm" (at 168.91 133.35 0)
-      (effects (font (size 1.27 1.27)) (justify left) hide)
-    )
-    (property "ipc land pattern name" "QFN50P300X300X75-16" (at 168.91 135.89 0)
-      (effects (font (size 1.27 1.27)) (justify left) hide)
-    )
-    (property "lead free" "Yes" (at 168.91 138.43 0)
-      (effects (font (size 1.27 1.27)) (justify left) hide)
-    )
-    (property "library id" "f761d93c558e3979" (at 168.91 140.97 0)
-      (effects (font (size 1.27 1.27)) (justify left) hide)
-    )
-    (property "max junction temp" "+150°C" (at 168.91 146.05 0)
-      (effects (font (size 1.27 1.27)) (justify left) hide)
-    )
-    (property "max supply voltage" "5.5V" (at 168.91 148.59 0)
-      (effects (font (size 1.27 1.27)) (justify left) hide)
-    )
-    (property "min supply voltage" "2.5V" (at 168.91 151.13 0)
-      (effects (font (size 1.27 1.27)) (justify left) hide)
-    )
-    (property "mouser part number" "700-MAX98357AETE+T" (at 168.91 153.67 0)
-      (effects (font (size 1.27 1.27)) (justify left) hide)
-    )
-    (property "nominal supply current" "2.4-2.75mA" (at 168.91 156.21 0)
-      (effects (font (size 1.27 1.27)) (justify left) hide)
-    )
-    (property "number of channels" "1" (at 168.91 158.75 0)
-      (effects (font (size 1.27 1.27)) (justify left) hide)
-    )
     (property "package" "TQFN16" (at 168.91 161.29 0)
       (effects (font (size 1.27 1.27)) (justify left) hide)
     )
-    (property "rohs" "Yes" (at 168.91 166.37 0)
-      (effects (font (size 1.27 1.27)) (justify left) hide)
-    )
-    (property "standoff height" "0mm" (at 168.91 168.91 0)
-      (effects (font (size 1.27 1.27)) (justify left) hide)
-    )
-    (property "temperature range high" "+85°C" (at 168.91 171.45 0)
-      (effects (font (size 1.27 1.27)) (justify left) hide)
-    )
-    (property "temperature range low" "-40°C" (at 168.91 173.99 0)
-      (effects (font (size 1.27 1.27)) (justify left) hide)
-    )
     (property "JLCPCB Part #" "C910544" (at 168.91 97.79 0)
       (effects (font (size 1.27 1.27)) hide)
@@
       (effects (font (size 1.27 1.27)) hide)
     )
-    (property "Substitution Comments" "Need to keep this compatible." (at 168.91 97.79 0)
-      (effects (font (size 1.27 1.27)) hide)
-    )
     (property "Manufacturer_Part_Number" "MAX98357AETE+T " (at 168.91 97.79 0)
       (effects (font (size 1.27 1.27)) hide)
     )
     (property "Mouser Part Number" "700-MAX98357AETE+T" (at 168.91 97.79 0)
+      (effects (font (size 1.27 1.27)) hide)
+    )
+    (property "MPN" "MAX98357AETE+T " (at 168.91 97.79 0)
       (effects (font (size 1.27 1.27)) hide)
     )
@@
   )
   (symbol (lib_id "Connector:Conn_01x02_Socket") (at 87.63 99.06 180) (unit 1)
-    (in_bom no) (on_board yes) (dnp no)
+    (in_bom no) (on_board yes) (dnp yes)
     (property "Reference" "J2" (at 88.265 92.71 0)
       (effects (font (size 1.27 1.27)))
@@
     )
     (property "Datasheet" "~" (at 87.63 99.06 0)
+      (effects (font (size 1.27 1.27)) hide)
+    )
+    (property "MPN" "" (at 87.63 99.06 0)
       (effects (font (size 1.27 1.27)) hide)
     )
@@
       (effects (font (size 1.27 1.27)) hide)
     )
-    (property "Substitution Comments" "Keep the value correct." (at 161.29 107.95 0)
-      (effects (font (size 1.27 1.27)) hide)
-    )
     (property "Manufacturer" "Murata" (at 161.29 107.95 0)
       (effects (font (size 1.27 1.27)) hide)
@@
     )
     (property "digikey part number" "490-GRM155R60J106ME05DTR-ND" (at 161.29 107.95 0)
+      (effects (font (size 1.27 1.27)) hide)
+    )
+    (property "package" "0402" (at 161.29 107.95 0)
+      (effects (font (size 1.27 1.27)) hide)
+    )
+    (property "MPN" "GRM155R60J106ME05D" (at 161.29 107.95 0)
       (effects (font (size 1.27 1.27)) hide)
     )
@@
       (effects (font (size 1.27 1.27)) hide)
     )
-    (property "Substitution Comments" "Keep the value correct." (at 171.45 93.98 0)
-      (effects (font (size 1.27 1.27)) hide)
-    )
     (property "Manufacturer" "TE Connectivity" (at 171.45 93.98 0)
       (effects (font (size 1.27 1.27)) hide)
@@
     )
     (property "digikey part number" "A130391TR-ND" (at 171.45 93.98 0)
+      (effects (font (size 1.27 1.27)) hide)
+    )
+    (property "package" "0402" (at 171.45 93.98 0)
+      (effects (font (size 1.27 1.27)) hide)
+    )
+    (property "MPN" "CRGP0402F1M0" (at 171.45 93.98 0)
       (effects (font (size 1.27 1.27)) hide)
     )
@@
       (effects (font (size 1.27 1.27)) hide)
     )
-    (property "Substitution Comments" "Keep the value correct." (at 100.33 83.82 0)
-      (effects (font (size 1.27 1.27)) hide)
-    )
     (property "Manufacturer" "Wurth Elektronik " (at 100.33 83.82 0)
       (effects (font (size 1.27 1.27)) hide)
@@
     )
     (property "digikey part number" "732-8048-2-ND" (at 100.33 83.82 0)
+      (effects (font (size 1.27 1.27)) hide)
+    )
+    (property "package" "0805" (at 100.33 83.82 0)
+      (effects (font (size 1.27 1.27)) hide)
+    )
+    (property "MPN" "885012207056 " (at 100.33 83.82 0)
       (effects (font (size 1.27 1.27)) hide)
     )
@@
       (effects (font (size 1.27 1.27)) hide)
     )
-    (property "MPN" "HCB1608KF-102T10" (at 116.84 100.33 0)
-      (effects (font (size 1.27 1.27)) hide)
-    )
     (property "Manufacturer" "Bourns" (at 116.84 100.33 0)
       (effects (font (size 1.27 1.27)) hide)
     )
-    (property "Substitution Comments" "Just make sure it can handle 1A. It's for a low-pass filter in analog audio output." (at 116.84 100.33 0)
-      (effects (font (size 1.27 1.27)) hide)
-    )
     (property "Manufacturer_Part_Number" "MH1608-471Y" (at 116.84 100.33 0)
       (effects (font (size 1.27 1.27)) hide)
@@
       (effects (font (size 1.27 1.27)) hide)
     )
+    (property "package" "0603" (at 116.84 100.33 0)
+      (effects (font (size 1.27 1.27)) hide)
+    )
+    (property "MPN" "MH1608-471Y" (at 116.84 100.33 0)
+      (effects (font (size 1.27 1.27)) hide)
+    )
