File: system-board/led-out.kicad_sch (KiCad schematic)
At the start: 8 parts, among them J5 BLADE_1, J6 BLADE_2, J7 BLADE_3, J8 BLADE_4, Q5 PMZB290UNE2YL

Commit message: First attempt
Parts:
- removed J5: BLADE_1, Connector_JST:JST_SH_SM02B-SRSS-TB_1x02-1MP_P1.00mm_Horizontal, symbol Connector:Conn_01x02_Socket
- removed J6: BLADE_2, Connector_JST:JST_SH_SM02B-SRSS-TB_1x02-1MP_P1.00mm_Horizontal, symbol Connector:Conn_01x02_Socket
- removed J7: BLADE_3, Connector_JST:JST_SH_SM02B-SRSS-TB_1x02-1MP_P1.00mm_Horizontal, symbol Connector:Conn_01x02_Socket
- removed J8: BLADE_4, Connector_JST:JST_SH_SM02B-SRSS-TB_1x02-1MP_P1.00mm_Horizontal, symbol Connector:Conn_01x02_Socket
- added J2: LEDs, Connector_PinSocket_2.00mm:PinSocket_2x04_P2.00mm_Vertical, symbol Connector_Generic:Conn_02x04_Odd_Even
Connections:
- net Blade_1_Out: now also J2.1 (Pin_1)
- net Blade_2_Out: now also J2.3 (Pin_3)
- net Blade_3_Out: now also J2.5 (Pin_5)
- net Blade_4_Out: now also J2.7 (Pin_7)
- net VDD: now also J2.2 (Pin_2), J2.4 (Pin_4), J2.6 (Pin_6), J2.8 (Pin_8)

Commit message: Redo system-board PCB to use fewer connectors
Parts:
- Q5: digikey part number (none) -> 1727-2328-2-ND
Changed lines of the file:
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@@
+      (effects (font (size 1.27 1.27)) hide)
+    )
+    (property "digikey part number" "1727-2328-2-ND" (at 179.07 78.74 0)
       (effects (font (size 1.27 1.27)) hide)
     )
@@
     )
     (property "Mouser Part Number" "771-PMZB290UNE2YL " (at 88.9 78.74 0)
+      (effects (font (size 1.27 1.27)) hide)
+    )
+    (property "digikey part number" "1727-2328-2-ND" (at 88.9 78.74 0)
       (effects (font (size 1.27 1.27)) hide)
     )
@@
       (effects (font (size 1.27 1.27)) hide)
     )
+    (property "digikey part number" "1727-2328-2-ND" (at 148.59 78.74 0)
+      (effects (font (size 1.27 1.27)) hide)
+    )
     (pin "1")
     (pin "2")
@@
       (effects (font (size 1.27 1.27)) hide)
     )
+    (property "digikey part number" "1727-2328-2-ND" (at 119.38 78.74 0)
+      (effects (font (size 1.27 1.27)) hide)
+    )

Commit message: Yet another PCB Revision
Parts:
- J2: now not fitted
- Q5: MPN (none) -> PMZB290UNE2YL; package (none) -> SOT-883-3
Changed lines of the file:
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@@
+      (effects (font (size 1.27 1.27)) hide)
+    )
+    (property "package" "SOT-883-3" (at 179.07 78.74 0)
+      (effects (font (size 1.27 1.27)) hide)
+    )
+    (property "MPN" "PMZB290UNE2YL" (at 179.07 78.74 0)
       (effects (font (size 1.27 1.27)) hide)
     )
@@
       (effects (font (size 1.27 1.27)) hide)
     )
+    (property "package" "SOT-883-3" (at 88.9 78.74 0)
+      (effects (font (size 1.27 1.27)) hide)
+    )
+    (property "MPN" "PMZB290UNE2YL" (at 88.9 78.74 0)
+      (effects (font (size 1.27 1.27)) hide)
+    )
     (pin "1")
     (pin "2")
@@
   )
   (symbol (lib_id "Connector_Generic:Conn_02x04_Odd_Even") (at 135.89 36.83 90) (unit 1)
-    (in_bom no) (on_board yes) (dnp no)
+    (in_bom no) (on_board yes) (dnp yes)
     (property "Reference" "J2" (at 143.51 34.29 90)
       (effects (font (size 1.27 1.27)) (justify right))
@@
     )
     (property "Datasheet" "~" (at 135.89 36.83 0)
+      (effects (font (size 1.27 1.27)) hide)
+    )
+    (property "MPN" "" (at 135.89 36.83 0)
       (effects (font (size 1.27 1.27)) hide)
     )
@@
       (effects (font (size 1.27 1.27)) hide)
     )
+    (property "package" "SOT-883-3" (at 148.59 78.74 0)
+      (effects (font (size 1.27 1.27)) hide)
+    )
+    (property "MPN" "PMZB290UNE2YL" (at 148.59 78.74 0)
+      (effects (font (size 1.27 1.27)) hide)
+    )
     (pin "1")
     (pin "2")
@@
       (effects (font (size 1.27 1.27)) hide)
     )
+    (property "package" "SOT-883-3" (at 119.38 78.74 0)
+      (effects (font (size 1.27 1.27)) hide)
+    )
+    (property "MPN" "PMZB290UNE2YL" (at 119.38 78.74 0)
+      (effects (font (size 1.27 1.27)) hide)
+    )

Commit message: Redo design again
Parts:
- renumbered J2 to J5
Changed lines of the file:
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@@
   (symbol (lib_id "Connector_Generic:Conn_02x04_Odd_Even") (at 135.89 36.83 90) (unit 1)
     (in_bom no) (on_board yes) (dnp yes)
-    (property "Reference" "J2" (at 143.51 34.29 90)
+    (property "Reference" "J5" (at 143.51 34.29 90)
       (effects (font (size 1.27 1.27)) (justify right))
     )
@@
       (project "system-board"
         (path "/54f22c46-3801-43f0-a916-fc0a05246fe7/37608a45-a840-496a-a0be-d1b7908a9637"
-          (reference "J2") (unit 1)
+          (reference "J5") (unit 1)
         )
       )
@@
   (symbol (lib_id "power:GND") (at 181.61 101.6 0) (unit 1)
     (in_bom yes) (on_board yes) (dnp no) (fields_autoplaced)
-    (property "Reference" "#PWR057" (at 181.61 107.95 0)
+    (property "Reference" "#PWR047" (at 181.61 107.95 0)
       (effects (font (size 1.27 1.27)) hide)
     )
@@
       (project "system-board"
         (path "/54f22c46-3801-43f0-a916-fc0a05246fe7/37608a45-a840-496a-a0be-d1b7908a9637"
-          (reference "#PWR057") (unit 1)
+          (reference "#PWR047") (unit 1)
         )
       )
@@
   (symbol (lib_id "power:GND") (at 151.13 101.6 0) (unit 1)
     (in_bom yes) (on_board yes) (dnp no) (fields_autoplaced)
-    (property "Reference" "#PWR056" (at 151.13 107.95 0)
+    (property "Reference" "#PWR046" (at 151.13 107.95 0)
       (effects (font (size 1.27 1.27)) hide)
     )
@@
       (project "system-board"
         (path "/54f22c46-3801-43f0-a916-fc0a05246fe7/37608a45-a840-496a-a0be-d1b7908a9637"
-          (reference "#PWR056") (unit 1)
+          (reference "#PWR046") (unit 1)
         )
       )
@@
   (symbol (lib_id "power:VDD") (at 129.54 24.13 0) (unit 1)
     (in_bom yes) (on_board yes) (dnp no) (fields_autoplaced)
-    (property "Reference" "#PWR053" (at 129.54 27.94 0)
+    (property "Reference" "#PWR043" (at 129.54 27.94 0)
       (effects (font (size 1.27 1.27)) hide)
     )
@@
       (project "system-board"
         (path "/54f22c46-3801-43f0-a916-fc0a05246fe7/37608a45-a840-496a-a0be-d1b7908a9637"
-          (reference "#PWR053") (unit 1)
+          (reference "#PWR043") (unit 1)
         )
       )
@@
   (symbol (lib_id "power:GND") (at 121.92 101.6 0) (unit 1)
     (in_bom yes) (on_board yes) (dnp no) (fields_autoplaced)
-    (property "Reference" "#PWR055" (at 121.92 107.95 0)
+    (property "Reference" "#PWR045" (at 121.92 107.95 0)
       (effects (font (size 1.27 1.27)) hide)
     )
@@
       (project "system-board"
         (path "/54f22c46-3801-43f0-a916-fc0a05246fe7/37608a45-a840-496a-a0be-d1b7908a9637"
-          (reference "#PWR055") (unit 1)
+          (reference "#PWR045") (unit 1)
         )
       )
@@
   (symbol (lib_id "power:GND") (at 91.44 101.6 0) (unit 1)
     (in_bom yes) (on_board yes) (dnp no) (fields_autoplaced)
-    (property "Reference" "#PWR054" (at 91.44 107.95 0)
+    (property "Reference" "#PWR044" (at 91.44 107.95 0)
       (effects (font (size 1.27 1.27)) hide)
     )
@@
       (project "system-board"
         (path "/54f22c46-3801-43f0-a916-fc0a05246fe7/37608a45-a840-496a-a0be-d1b7908a9637"
-          (reference "#PWR054") (unit 1)
-        )
-      )
+          (reference "#PWR044") (unit 1)
+        )
+      )
