File: system-board/power.kicad_sch (KiCad schematic)
At the start: 26 parts, among them IC2 AP2115M-3.3TRG1, Q1 DMP1012UFDF, Q2 SSM6K504NU.LF, Q3 SSM6K504NU.LF, Q4 DMP1012UFDF, U3 BQ29705DSER, U4 MCP73832-2-OT

Commit message: Redo system-board PCB to use fewer connectors
Parts:
- removed IC2: AP2115M-3.3TRG1, Package_SO:SOIC-8_3.9x4.9mm_P1.27mm, symbol imports:AP2115M-3.3TRG1
- removed U4: MCP73832-2-OT, Package_TO_SOT_SMD:SOT-23-5, symbol Battery_Management:MCP73832-2-OT
- added IC3: NCP186AMX330TAG, Imports:NCP186AMX330TAG, symbol imports:NCP186AMX330TAG
- added IC4: MCP73834T-FCI_MF, Imports:SON50P300X300X100-11N-D, symbol imports:MCP73834T-FCI_MF
- added R17: 10k, Resistor_SMD:R_0402_1005Metric, symbol Device:R_Small_US
- C10: digikey part number (none) -> 478-KGM03AR50J104KHTR-ND
- C12, C8: digikey part number (none) -> 1276-1907-2-ND
- C15, C9: digikey part number (none) -> 490-GRM155R60J106ME05DTR-ND
- D5: digikey part number (none) -> 160-1830-2-ND
- D6: value RSX501LAM20TR -> PMEG1030EJ; footprint Imports:SODFL4725X105N -> Diode_SMD:D_SOD-323F; Height 1.05 -> (none); JLCPCB Part # C253526 -> C133633; Manufacturer ROHM Semicon -> Nexperia; Manufacturer_Name ROHM Semiconductor -> Nexperia; Manufacturer_Part_Number RSX501LAM20TR -> PMEG1030EJ,115; Mouser Part Number 755-RSX501LAM20TR -> 771-PMEG1030EJ-T/R; Mouser Price/Stock https://www.mouser.co.uk/ProductDetail/ROHM-Semiconductor/R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 -> (none); digikey part number (none) -> 1727-3852-2-ND
- Q1, Q4: digikey part number (none) -> DMP1012UFDF-7-ND
- Q2, Q3: digikey part number (none) -> SSM6K504NULFTR-ND
- R10: digikey part number (none) -> A121534TR-ND
- R11: digikey part number (none) -> 311-2.0KJRTR-ND
- R12: digikey part number (none) -> 311-200LRTR-ND
- R8, R9: digikey part number (none) -> 541-3971-2-ND
- U3: JLCPCB Part # (none) -> C2876296; Manufacturer (none) -> Texas Instruments; Manufacturer_Part_Number (none) -> BQ29705DSER; Mouser Part Number (none) -> 595-BQ29705DSER; digikey part number (none) -> 296-39946-2-ND
Connections:
- net BATT_PROT_+: now also IC4.10 (VBAT_2), IC4.9 (VBAT_1)
- net CHARGING: now also IC4.3 (STAT1)
- net GND: now also IC3.5 (GND_1), IC3.9 (GND_2), IC4.11 (EP), IC4.5 (VSS), IC4.7 (~{PG_(}TE)), R17.2
- net VBUS: now also IC4.1 (VDD_1), IC4.2 (VDD_2)
- net VCC: now also IC3.1 (OUT_1), IC3.2 (OUT_2), IC3.4 (FB)
- net VDD: now also IC3.7 (IN_1), IC3.8 (IN_2)
- net VREG_EN: now reaches R15.2
- net VREG_EN: now also IC3.6 (EN)
- net at R11.1: now also IC4.6 (PROG)
- net BATT_FILTERED: now reaches C10.1, R8.2, U3.5 (BAT)
- new net: IC4.8 (THERM), R17.1
- no-connect marks 3 -> 1
Other:
- moved on the sheet: C12, C9, R11, R15, R8

Commit message: Yet another PCB Revision
Parts:
- C10: MPN (none) -> 02016D104KAT2A; Manufacturer 02016D104KAT2A -> Kyocera AVX; package (none) -> 0201
- C12, C8: MPN (none) -> CL10A475MQ8NNNC; package (none) -> 0603
- C15, C9: MPN (none) -> GRM155R60J106ME05D; package (none) -> 0402
- D4: MPN (none) -> BZX38450-C1V8X; package (none) -> SOD-323
- D5: MPN (none) -> LTST-C193KRKT-5A; package (none) -> 0603
- D6: MPN (none) -> PMEG1030EJ,115; Manufacturer_Name Nexperia -> (none); package (none) -> SOD-323
- IC3: Height 0 -> (none); MPN (none) -> NCP186AMX330TAG; Manufacturer_Name onsemi -> (none); package (none) -> DFN-8-EP(1.2x1.6)
- IC4: Height 1 -> (none); MPN (none) -> MCP73834T-FCI/MF; Manufacturer_Name Microchip -> (none); package (none) -> DFN-10-EP(3x3)
- Q1, Q4: JLCPCB Part # (none) -> C5245345; MPN (none) -> DMP1012UFDF-7; package (none) -> U-DFN2020-6
- Q2, Q3: MPN (none) -> SSM6K504NU,LF; package (none) -> UDFN-6(2x2)
- R10: MPN (none) -> CRG0402F1K0; package (none) -> 0402
- R11: MPN (none) -> RC0402JR-072KL; package (none) -> 0402
- R12: MPN (none) -> RC0402FR-07200RL; package (none) -> 0402
- R13, R14, R15, R16: MPN (none) -> RMC10K104FTH; package (none) -> 0402
- R17: MPN (none) -> RC0402JR-075K1P; package (none) -> 0402
- R8: MPN (none) -> RMC10-331JTH; package (none) -> 0402
- R9: MPN (none) -> CRCW04022K20FKEDC; package (none) -> 0402
- U3: MPN (none) -> BQ29705DSER; package (none) -> DFN-6(1.5x1.5)

Commit message: Redo design again
Parts:
- removed IC3: NCP186AMX330TAG, Imports:NCP186AMX330TAG, symbol imports:NCP186AMX330TAG
- added U4: TLV75733PDRV, Package_SON:WSON-6-1EP_2x2mm_P0.65mm_EP1x1.6mm, symbol Regulator_Linear:TLV75733PDRV
- C10: footprint Capacitor_SMD:C_0201_0603Metric -> Capacitor_SMD:C_0402_1005Metric; JLCPCB Part # C5188607 -> C60474; MPN 02016D104KAT2A -> CC0402KRX7R7BB104; Manufacturer Kyocera AVX -> YAGEO; Manufacturer_Part_Number 02016D104KAT2A -> CC0402KRX7R7BB104; Mouser Part Number 581-02016D104KAT2A -> 603-CC402KRX7R7BB104; digikey part number 478-KGM03AR50J104KHTR-ND -> 311-1338-6-ND; package 0201 -> 0402
- C12: footprint Capacitor_SMD:C_0603_1608Metric -> Capacitor_SMD:C_0402_1005Metric; JLCPCB Part # C154959 -> C368809; MPN CL10A475MQ8NNNC -> CL05A475KP5NRNC; Manufacturer_Part_Number CL10A475MQ8NNNC -> CL05A475KP5NRNC; Mouser Part Number 187-CL10A475MQ8NNNC -> 187-CL05A475KP5NRNC; digikey part number 1276-1907-2-ND -> 1276-1480-6-ND; package 0603 -> 0402
- C8: footprint Capacitor_SMD:C_0603_1608Metric -> Capacitor_SMD:C_0402_1005Metric; JLCPCB Part # C154959 -> C368809; MPN CL10A475MQ8NNNC -> CL05A475KP5NRNC; Manufacturer_Part_Number CL10A475MQ8NNNC -> CC0402MRX5R5BB475; Mouser Part Number 187-CL10A475MQ8NNNC -> 187-CL05A475KP5NRNC; digikey part number 1276-1907-2-ND -> 1276-1480-6-ND; package 0603 -> 0402
- R9: renamed from R17; Mouser Part Number RC0402JR-075K1P -> 603-RC0402JR-075K1P
- renumbered C15 to C13, IC4 to IC2, R12 to R11, R13 to R12, R14 to R13, R16 to R14, R8 to R6, R9 to R7, R11 to R8
Connections:
- net VREG_EN is gone; now on net VDD: R15.2
- net GND: now also U4.3 (GND), U4.7 (GND)
- net VCC: now also U4.1 (OUT)
- net VDD: now also U4.6 (IN); no longer R15.1
- new net: R15.1, U4.4 (EN)
Other:
- moved on the sheet: C12, C8
